File: IO4-IR-Detector-Active-Mount_array.brd (EAGLE design)
At the start: 114.3 x 116.8 mm, 43 parts

Commit message: added values for connectors
Parts:
- JP1X11, JP1X12, JP1X13, JP1X21, JP1X22, JP1X23, JP1X31, JP1X32, JP1X33, JP1X41, JP1X42, JP1X43, JP1X51, JP1X52, JP1X53, JP1X61, JP1X62, JP1X63, JP1X71, JP1X72, JP1X73: value (none) -> 0.100
Changed lines of the file:
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@@
 </autorouter>
 <elements>
-<element name="JP1X11" library="SPCoast" package="1X04_LOCK" value="" x="7.62" y="28.575"/>
+<element name="JP1X11" library="SPCoast" package="1X04_LOCK" value="0.100" x="7.62" y="28.575"/>
 <element name="PD1X11" library="SPCoast" package="RPR220" value="" x="11.43" y="33.655"/>
-<element name="JP1X12" library="SPCoast" package="1X04_LOCK" value="" x="7.62" y="53.975"/>
+<element name="JP1X12" library="SPCoast" package="1X04_LOCK" value="0.100" x="7.62" y="53.975"/>
 <element name="PD1X12" library="SPCoast" package="RPR220" value="" x="11.43" y="59.055"/>
-<element name="JP1X13" library="SPCoast" package="1X04_LOCK" value="" x="7.62" y="79.375"/>
+<element name="JP1X13" library="SPCoast" package="1X04_LOCK" value="0.100" x="7.62" y="79.375"/>
 <element name="PD1X13" library="SPCoast" package="RPR220" value="" x="11.43" y="84.455"/>
-<element name="JP1X21" library="SPCoast" package="1X04_LOCK" value="" x="20.32" y="28.575"/>
+<element name="JP1X21" library="SPCoast" package="1X04_LOCK" value="0.100" x="20.32" y="28.575"/>
 <element name="PD1X21" library="SPCoast" package="RPR220" value="" x="24.13" y="33.655"/>
-<element name="JP1X22" library="SPCoast" package="1X04_LOCK" value="" x="20.32" y="53.975"/>
+<element name="JP1X22" library="SPCoast" package="1X04_LOCK" value="0.100" x="20.32" y="53.975"/>
 <element name="PD1X22" library="SPCoast" package="RPR220" value="" x="24.13" y="59.055"/>
-<element name="JP1X23" library="SPCoast" package="1X04_LOCK" value="" x="20.32" y="79.375"/>
+<element name="JP1X23" library="SPCoast" package="1X04_LOCK" value="0.100" x="20.32" y="79.375"/>
 <element name="PD1X23" library="SPCoast" package="RPR220" value="" x="24.13" y="84.455"/>
-<element name="JP1X31" library="SPCoast" package="1X04_LOCK" value="" x="33.02" y="28.575"/>
+<element name="JP1X31" library="SPCoast" package="1X04_LOCK" value="0.100" x="33.02" y="28.575"/>
 <element name="PD1X31" library="SPCoast" package="RPR220" value="" x="36.83" y="33.655"/>
-<element name="JP1X32" library="SPCoast" package="1X04_LOCK" value="" x="33.02" y="53.975"/>
+<element name="JP1X32" library="SPCoast" package="1X04_LOCK" value="0.100" x="33.02" y="53.975"/>
 <element name="PD1X32" library="SPCoast" package="RPR220" value="" x="36.83" y="59.055"/>
-<element name="JP1X33" library="SPCoast" package="1X04_LOCK" value="" x="33.02" y="79.375"/>
+<element name="JP1X33" library="SPCoast" package="1X04_LOCK" value="0.100" x="33.02" y="79.375"/>
 <element name="PD1X33" library="SPCoast" package="RPR220" value="" x="36.83" y="84.455"/>
-<element name="JP1X41" library="SPCoast" package="1X04_LOCK" value="" x="45.72" y="28.575"/>
+<element name="JP1X41" library="SPCoast" package="1X04_LOCK" value="0.100" x="45.72" y="28.575"/>
 <element name="PD1X41" library="SPCoast" package="RPR220" value="" x="49.53" y="33.655"/>
-<element name="JP1X42" library="SPCoast" package="1X04_LOCK" value="" x="45.72" y="53.975"/>
+<element name="JP1X42" library="SPCoast" package="1X04_LOCK" value="0.100" x="45.72" y="53.975"/>
 <element name="PD1X42" library="SPCoast" package="RPR220" value="" x="49.53" y="59.055"/>
-<element name="JP1X43" library="SPCoast" package="1X04_LOCK" value="" x="45.72" y="79.375"/>
+<element name="JP1X43" library="SPCoast" package="1X04_LOCK" value="0.100" x="45.72" y="79.375"/>
 <element name="PD1X43" library="SPCoast" package="RPR220" value="" x="49.53" y="84.455"/>
-<element name="JP1X51" library="SPCoast" package="1X04_LOCK" value="" x="58.42" y="28.575"/>
+<element name="JP1X51" library="SPCoast" package="1X04_LOCK" value="0.100" x="58.42" y="28.575"/>
 <element name="PD1X51" library="SPCoast" package="RPR220" value="" x="62.23" y="33.655"/>
-<element name="JP1X52" library="SPCoast" package="1X04_LOCK" value="" x="58.42" y="53.975"/>
+<element name="JP1X52" library="SPCoast" package="1X04_LOCK" value="0.100" x="58.42" y="53.975"/>
 <element name="PD1X52" library="SPCoast" package="RPR220" value="" x="62.23" y="59.055"/>
-<element name="JP1X53" library="SPCoast" package="1X04_LOCK" value="" x="58.42" y="79.375"/>
+<element name="JP1X53" library="SPCoast" package="1X04_LOCK" value="0.100" x="58.42" y="79.375"/>
 <element name="PD1X53" library="SPCoast" package="RPR220" value="" x="62.23" y="84.455"/>
-<element name="JP1X61" library="SPCoast" package="1X04_LOCK" value="" x="71.12" y="28.575"/>
+<element name="JP1X61" library="SPCoast" package="1X04_LOCK" value="0.100" x="71.12" y="28.575"/>
 <element name="PD1X61" library="SPCoast" package="RPR220" value="" x="74.93" y="33.655"/>
-<element name="JP1X62" library="SPCoast" package="1X04_LOCK" value="" x="71.12" y="53.975"/>
+<element name="JP1X62" library="SPCoast" package="1X04_LOCK" value="0.100" x="71.12" y="53.975"/>
 <element name="PD1X62" library="SPCoast" package="RPR220" value="" x="74.93" y="59.055"/>
-<element name="JP1X63" library="SPCoast" package="1X04_LOCK" value="" x="71.12" y="79.375"/>
+<element name="JP1X63" library="SPCoast" package="1X04_LOCK" value="0.100" x="71.12" y="79.375"/>
 <element name="PD1X63" library="SPCoast" package="RPR220" value="" x="74.93" y="84.455"/>
-<element name="JP1X71" library="SPCoast" package="1X04_LOCK" value="" x="83.82" y="28.575"/>
+<element name="JP1X71" library="SPCoast" package="1X04_LOCK" value="0.100" x="83.82" y="28.575"/>
 <element name="PD1X71" library="SPCoast" package="RPR220" value="" x="87.63" y="33.655"/>
-<element name="JP1X72" library="SPCoast" package="1X04_LOCK" value="" x="83.82" y="53.975"/>
+<element name="JP1X72" library="SPCoast" package="1X04_LOCK" value="0.100" x="83.82" y="53.975"/>
 <element name="PD1X72" library="SPCoast" package="RPR220" value="" x="87.63" y="59.055"/>
-<element name="JP1X73" library="SPCoast" package="1X04_LOCK" value="" x="83.82" y="79.375"/>
+<element name="JP1X73" library="SPCoast" package="1X04_LOCK" value="0.100" x="83.82" y="79.375"/>
 <element name="PD1X73" library="SPCoast" package="RPR220" value="" x="87.63" y="84.455"/>
 <element name="PD1X1" library="SPCoast" package="BOARD-SEEED10X10-NOHOLES" value="" x="0" y="0"/>

Commit message: added values for connectors
Parts:
- PD1X11, PD1X12, PD1X13, PD1X21, PD1X22, PD1X23, PD1X31, PD1X32, PD1X33, PD1X41, PD1X42, PD1X43, PD1X51, PD1X52, PD1X53, PD1X61, PD1X62, PD1X63, PD1X71, PD1X72, PD1X73: value (none) -> RPR220
Changed lines of the file:
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@@
 <elements>
 <element name="JP1X11" library="SPCoast" package="1X04_LOCK" value="0.100" x="7.62" y="28.575"/>
-<element name="PD1X11" library="SPCoast" package="RPR220" value="" x="11.43" y="33.655"/>
+<element name="PD1X11" library="SPCoast" package="RPR220" value="RPR220" x="11.43" y="33.655"/>
 <element name="JP1X12" library="SPCoast" package="1X04_LOCK" value="0.100" x="7.62" y="53.975"/>
-<element name="PD1X12" library="SPCoast" package="RPR220" value="" x="11.43" y="59.055"/>
+<element name="PD1X12" library="SPCoast" package="RPR220" value="RPR220" x="11.43" y="59.055"/>
 <element name="JP1X13" library="SPCoast" package="1X04_LOCK" value="0.100" x="7.62" y="79.375"/>
-<element name="PD1X13" library="SPCoast" package="RPR220" value="" x="11.43" y="84.455"/>
+<element name="PD1X13" library="SPCoast" package="RPR220" value="RPR220" x="11.43" y="84.455"/>
 <element name="JP1X21" library="SPCoast" package="1X04_LOCK" value="0.100" x="20.32" y="28.575"/>
-<element name="PD1X21" library="SPCoast" package="RPR220" value="" x="24.13" y="33.655"/>
+<element name="PD1X21" library="SPCoast" package="RPR220" value="RPR220" x="24.13" y="33.655"/>
 <element name="JP1X22" library="SPCoast" package="1X04_LOCK" value="0.100" x="20.32" y="53.975"/>
-<element name="PD1X22" library="SPCoast" package="RPR220" value="" x="24.13" y="59.055"/>
+<element name="PD1X22" library="SPCoast" package="RPR220" value="RPR220" x="24.13" y="59.055"/>
 <element name="JP1X23" library="SPCoast" package="1X04_LOCK" value="0.100" x="20.32" y="79.375"/>
-<element name="PD1X23" library="SPCoast" package="RPR220" value="" x="24.13" y="84.455"/>
+<element name="PD1X23" library="SPCoast" package="RPR220" value="RPR220" x="24.13" y="84.455"/>
 <element name="JP1X31" library="SPCoast" package="1X04_LOCK" value="0.100" x="33.02" y="28.575"/>
-<element name="PD1X31" library="SPCoast" package="RPR220" value="" x="36.83" y="33.655"/>
+<element name="PD1X31" library="SPCoast" package="RPR220" value="RPR220" x="36.83" y="33.655"/>
 <element name="JP1X32" library="SPCoast" package="1X04_LOCK" value="0.100" x="33.02" y="53.975"/>
-<element name="PD1X32" library="SPCoast" package="RPR220" value="" x="36.83" y="59.055"/>
+<element name="PD1X32" library="SPCoast" package="RPR220" value="RPR220" x="36.83" y="59.055"/>
 <element name="JP1X33" library="SPCoast" package="1X04_LOCK" value="0.100" x="33.02" y="79.375"/>
-<element name="PD1X33" library="SPCoast" package="RPR220" value="" x="36.83" y="84.455"/>
+<element name="PD1X33" library="SPCoast" package="RPR220" value="RPR220" x="36.83" y="84.455"/>
 <element name="JP1X41" library="SPCoast" package="1X04_LOCK" value="0.100" x="45.72" y="28.575"/>
-<element name="PD1X41" library="SPCoast" package="RPR220" value="" x="49.53" y="33.655"/>
+<element name="PD1X41" library="SPCoast" package="RPR220" value="RPR220" x="49.53" y="33.655"/>
 <element name="JP1X42" library="SPCoast" package="1X04_LOCK" value="0.100" x="45.72" y="53.975"/>
-<element name="PD1X42" library="SPCoast" package="RPR220" value="" x="49.53" y="59.055"/>
+<element name="PD1X42" library="SPCoast" package="RPR220" value="RPR220" x="49.53" y="59.055"/>
 <element name="JP1X43" library="SPCoast" package="1X04_LOCK" value="0.100" x="45.72" y="79.375"/>
-<element name="PD1X43" library="SPCoast" package="RPR220" value="" x="49.53" y="84.455"/>
+<element name="PD1X43" library="SPCoast" package="RPR220" value="RPR220" x="49.53" y="84.455"/>
 <element name="JP1X51" library="SPCoast" package="1X04_LOCK" value="0.100" x="58.42" y="28.575"/>
-<element name="PD1X51" library="SPCoast" package="RPR220" value="" x="62.23" y="33.655"/>
+<element name="PD1X51" library="SPCoast" package="RPR220" value="RPR220" x="62.23" y="33.655"/>
 <element name="JP1X52" library="SPCoast" package="1X04_LOCK" value="0.100" x="58.42" y="53.975"/>
-<element name="PD1X52" library="SPCoast" package="RPR220" value="" x="62.23" y="59.055"/>
+<element name="PD1X52" library="SPCoast" package="RPR220" value="RPR220" x="62.23" y="59.055"/>
 <element name="JP1X53" library="SPCoast" package="1X04_LOCK" value="0.100" x="58.42" y="79.375"/>
-<element name="PD1X53" library="SPCoast" package="RPR220" value="" x="62.23" y="84.455"/>
+<element name="PD1X53" library="SPCoast" package="RPR220" value="RPR220" x="62.23" y="84.455"/>
 <element name="JP1X61" library="SPCoast" package="1X04_LOCK" value="0.100" x="71.12" y="28.575"/>
-<element name="PD1X61" library="SPCoast" package="RPR220" value="" x="74.93" y="33.655"/>
+<element name="PD1X61" library="SPCoast" package="RPR220" value="RPR220" x="74.93" y="33.655"/>
 <element name="JP1X62" library="SPCoast" package="1X04_LOCK" value="0.100" x="71.12" y="53.975"/>
-<element name="PD1X62" library="SPCoast" package="RPR220" value="" x="74.93" y="59.055"/>
+<element name="PD1X62" library="SPCoast" package="RPR220" value="RPR220" x="74.93" y="59.055"/>
 <element name="JP1X63" library="SPCoast" package="1X04_LOCK" value="0.100" x="71.12" y="79.375"/>
-<element name="PD1X63" library="SPCoast" package="RPR220" value="" x="74.93" y="84.455"/>
+<element name="PD1X63" library="SPCoast" package="RPR220" value="RPR220" x="74.93" y="84.455"/>
 <element name="JP1X71" library="SPCoast" package="1X04_LOCK" value="0.100" x="83.82" y="28.575"/>
-<element name="PD1X71" library="SPCoast" package="RPR220" value="" x="87.63" y="33.655"/>
+<element name="PD1X71" library="SPCoast" package="RPR220" value="RPR220" x="87.63" y="33.655"/>
 <element name="JP1X72" library="SPCoast" package="1X04_LOCK" value="0.100" x="83.82" y="53.975"/>
-<element name="PD1X72" library="SPCoast" package="RPR220" value="" x="87.63" y="59.055"/>
+<element name="PD1X72" library="SPCoast" package="RPR220" value="RPR220" x="87.63" y="59.055"/>
 <element name="JP1X73" library="SPCoast" package="1X04_LOCK" value="0.100" x="83.82" y="79.375"/>
-<element name="PD1X73" library="SPCoast" package="RPR220" value="" x="87.63" y="84.455"/>
+<element name="PD1X73" library="SPCoast" package="RPR220" value="RPR220" x="87.63" y="84.455"/>
 <element name="PD1X1" library="SPCoast" package="BOARD-SEEED10X10-NOHOLES" value="" x="0" y="0"/>
 </elements>

Commit message: added values for connectors
Parts:
- PD1X1: value (none) -> 10x10
Changed lines of the file:
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@@
 <element name="JP1X73" library="SPCoast" package="1X04_LOCK" value="0.100" x="83.82" y="79.375"/>
 <element name="PD1X73" library="SPCoast" package="RPR220" value="RPR220" x="87.63" y="84.455"/>
-<element name="PD1X1" library="SPCoast" package="BOARD-SEEED10X10-NOHOLES" value="" x="0" y="0"/>
+<element name="PD1X1" library="SPCoast" package="BOARD-SEEED10X10-NOHOLES" value="10x10" x="0" y="0"/>
 </elements>
 <signals>

Commit message: normalized values
Parts:
- PD1X1: value 10x10 -> BOARD
Changed lines of the file:
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@@
 <element name="JP1X73" library="SPCoast" package="1X04_LOCK" value="0.100" x="83.82" y="79.375"/>
 <element name="PD1X73" library="SPCoast" package="RPR220" value="RPR220" x="87.63" y="84.455"/>
-<element name="PD1X1" library="SPCoast" package="BOARD-SEEED10X10-NOHOLES" value="10x10" x="0" y="0"/>
+<element name="PD1X1" library="SPCoast" package="BOARD-SEEED10X10-NOHOLES" value="BOARD" x="0" y="0"/>
 </elements>
 <signals>
